File: PCB/Scratchpad.kicad_sch (KiCad schematic)
At the start: 52 parts, among them J1 USB_C_Receptacle_USB2.0, J2 I2C, J3 MIDI IN, J4 MIDI OUT, J5 OLED, SW1 Rotary_Encoder_Switch, SW10 SW_SPST, SW11 SW_SPST, SW12 SW_SPST, SW13 SW_SPST, SW14 SW_SPST, SW15 SW_SPST, SW16 SW_SPST, SW17 SW_SPST, SW18 SW_SPST, SW19 SW_SPST, SW2 Rotary_Encoder_Switch, SW20 SW_SPST, SW21 SW_SPST, SW22 SW_SPST, SW23 SW_SPST, SW24 SW_SPST, SW25 SW_SPST, SW26 Rotary_Encoder_Switch, SW3 Rotary_Encoder_Switch, SW4 Rotary_Encoder_Switch, SW5 SW_SPST, SW6 SW_SPST, SW7 SW_SPST, SW8 SW_SPST, SW9 SW_SPST, U1 COM-09032, U2 COM-09032, U3 RP2040TR7

Commit message: Added some components, I2C is pin header now
Parts:
- J2: footprint Keebio-Parts:TRRS_Jack -> Connector_PinHeader_2.54mm:PinHeader_1x04_P2.54mm_Vertical; symbol Connector:Conn_01x05_Female -> Connector:Conn_01x04_Female
- gave numbers to parts that had none: 1
Other:
- moved on the sheet: U1, U2, U3, U4

Commit message: Some footprint updates
Parts:
- J2: footprint Connector_PinHeader_2.54mm:PinHeader_1x04_P2.54mm_Vertical -> Connector_PinSocket_2.54mm:PinSocket_1x04_P2.54mm_Vertical
Changed lines of the file:
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@@
       (effects (font (size 1.27 1.27)) (justify left))
     )
-    (property "Footprint" "Connector_PinHeader_2.54mm:PinHeader_1x04_P2.54mm_Vertical" (id 2) (at 156.21 105.41 0)
+    (property "Footprint" "Connector_PinSocket_2.54mm:PinSocket_1x04_P2.54mm_Vertical" (id 2) (at 156.21 105.41 0)
       (effects (font (size 1.27 1.27)) hide)
     )
@@
     )
     (path "/2e4e5548-0c84-4d3e-a301-c17e153937b8"
-      (reference "J2") (unit 1) (value "I2C") (footprint "Connector_PinHeader_2.54mm:PinHeader_1x04_P2.54mm_Vertical")
+      (reference "J2") (unit 1) (value "I2C") (footprint "Connector_PinSocket_2.54mm:PinSocket_1x04_P2.54mm_Vertical")
     )
     (path "/d6691a51-8be0-424a-8ab6-9098936df2d1"
